File: 2-Hardware/egg_feather_brd.sch (KiCad schematic (older format))
At the start: 5 parts, among them SW1 SWITCH_SPST, U1 ADAFRUIT_FEATHER, U2 LIS3DH_BOB

Commit message: Moved part off pin 13 to pin 11
Moved part off pin 13, new part placement on board
Changed lines of the file:
@@
 LIBS:contrib
 LIBS:valves
-LIBS:MiscellaneousDevices
-LIBS:Sensors
 LIBS:egg_feather_brd-cache
 EELAYER 25 0
@@
 	1    0    0    -1
 $EndComp
-Wire Wire Line
-	5050 4250 6200 4250
-Wire Wire Line
-	6200 4250 6200 4550
-Wire Wire Line
-	6200 4550 6300 4550
 Wire Wire Line
 	5050 4700 6200 4700
@@
 	6000 5350 6300 5350
 Connection ~ 6150 2700
+Wire Wire Line
+	5050 4250 5200 4250
+Wire Wire Line
+	5200 4250 5200 4750
+Wire Wire Line
+	5200 4750 6300 4750
 $EndSCHEMATC

Commit message: Schematic update
Parts:
- D1, D2: footprint LEDs:LED_D5.0mm -> LEDs:LED_1206
Changed lines of the file:
@@
 LIBS:contrib
 LIBS:valves
+LIBS:Sensors
 LIBS:egg_feather_brd-cache
 EELAYER 25 0
@@
 F 0 "D2" H 4900 4800 50  0000 C CNN
 F 1 "LED" H 4900 4600 50  0000 C CNN
-F 2 "LEDs:LED_D5.0mm" H 4900 4700 50  0001 C CNN
+F 2 "LEDs:LED_1206" H 4900 4700 50  0001 C CNN
 F 3 "" H 4900 4700 50  0001 C CNN
 	1    4900 4700
@@
 F 0 "D1" H 4900 4350 50  0000 C CNN
 F 1 "LED" H 4900 4150 50  0000 C CNN
-F 2 "LEDs:LED_D5.0mm" H 4900 4250 50  0001 C CNN
+F 2 "LEDs:LED_1206" H 4900 4250 50  0001 C CNN
 F 3 "" H 4900 4250 50  0001 C CNN
 	1    4900 4250

Commit message: Updates for KiCad 5, routed board for test run
Parts:
- D1, D2: symbol LED -> Device:LED
- SW1: symbol SWITCH_SPST -> egg_feather_brd-rescue:SWITCH_SPST
- U1: symbol ADAFRUIT_FEATHER -> egg_feather_brd-rescue:ADAFRUIT_FEATHER
- U2: symbol LIS3DH_BOB -> egg_feather_brd-rescue:LIS3DH_BOB
Connections:
- wire segments 33 -> 36
Changed lines of the file:
@@
-EESchema Schematic File Version 2
-LIBS:power
-LIBS:device
-LIBS:transistors
-LIBS:conn
-LIBS:linear
-LIBS:regul
-LIBS:74xx
-LIBS:cmos4000
-LIBS:adc-dac
-LIBS:memory
-LIBS:xilinx
-LIBS:microcontrollers
-LIBS:dsp
-LIBS:microchip
-LIBS:analog_switches
-LIBS:motorola
-LIBS:texas
-LIBS:intel
-LIBS:audio
-LIBS:interface
-LIBS:digital-audio
-LIBS:philips
-LIBS:display
-LIBS:cypress
-LIBS:siliconi
-LIBS:opto
-LIBS:atmel
-LIBS:contrib
-LIBS:valves
-LIBS:Sensors
+EESchema Schematic File Version 4
 LIBS:egg_feather_brd-cache
-EELAYER 25 0
+EELAYER 26 0
 EELAYER END
 $Descr A4 11693 8268
@@
 $EndDescr
 $Comp
-L ADAFRUIT_FEATHER U1
+L egg_feather_brd-rescue:ADAFRUIT_FEATHER U1
 U 1 1 5955C01D
 P 6550 4800
@@
 $EndComp
 $Comp
-L ADAFRUIT_FEATHER U1
+L egg_feather_brd-rescue:ADAFRUIT_FEATHER U1
 U 2 1 5955C0DA
 P 6600 3150
@@
 $EndComp
 $Comp
-L LED D2
+L Device:LED D2
 U 1 1 5955CFB2
 P 4900 4700
@@
 $EndComp
 $Comp
-L LED D1
+L Device:LED D1
 U 1 1 5955D02F
 P 4900 4250
@@
 $EndComp
 $Comp
-L SWITCH_SPST SW1
+L egg_feather_brd-rescue:SWITCH_SPST SW1
 U 1 1 5955E018
 P 4900 5200
@@
 	4750 4250 4550 4250
 Wire Wire Line
-	4550 2700 4550 5200
+	4550 2700 4550 4250
 Wire Wire Line
 	4550 4700 4750 4700
@@
 Connection ~ 4550 4700
 $Comp
-L LIS3DH_BOB U2
+L egg_feather_brd-rescue:LIS3DH_BOB U2
 U 1 1 595FB4D9
 P 8750 3000
@@
 	6150 2100 6150 2700
 Wire Wire Line
-	4550 2700 6350 2700
+	4550 2700 6150 2700
 Wire Wire Line
 	8050 3300 7500 3300
@@
 Wire Wire Line
 	5200 4750 6300 4750
+Wire Wire Line
+	4550 4250 4550 4700
+Wire Wire Line
+	4550 4700 4550 5200
+Wire Wire Line
+	6150 2700 6350 2700
 $EndSCHEMATC
